File: UNO-128DA28.kicad_sch (KiCad schematic)
At the start: 55 parts, among them J1 USB_B, J2 Barrel_Jack_Switch, J3 PF0, J4 PF1, J5 Alternate pin 8, connection, J6 MODE, J7 GND, J8 UPDI_SEL, Q1 FDN340P, SW1 Reset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

Commit message: Updated all the files.
Credits added to the original idea people.
Parts:
- J5: value Alternate pin 8, connection -> Alternate pin 9, connection
Other:
- note added: "The upload mode is designed by Hans(MCUdude). Credits to idea of the original board idea go to Bill(WestfW)."
